File: $drawdio.sch (KiCad schematic (older format))
At the start: 12 parts, among them P1 CONN_2, Q1 BC558, Q2 BC547, U1 LM555N

Commit message: V0.2
Parts:
- P2: renamed from P?; footprint (none) -> Pin_Headers:Pin_Header_Straight_1x01
Changed lines of the file:
@@
 $EndComp
 $Comp
-L GND-RESCUE-drawdio #PWR06
+L GND-RESCUE-drawdio #PWR05
 U 1 1 553585E1
 P 3650 5050
-F 0 "#PWR06" H 3650 5050 30  0001 C CNN
+F 0 "#PWR05" H 3650 5050 30  0001 C CNN
 F 1 "GND" H 3650 4980 30  0001 C CNN
 F 2 "" H 3650 5050 60  0000 C CNN
@@
 $EndComp
 $Comp
-L VCC #PWR07
+L VCC #PWR06
 U 1 1 553585F0
 P 7400 3550
-F 0 "#PWR07" H 7400 3650 30  0001 C CNN
+F 0 "#PWR06" H 7400 3650 30  0001 C CNN
 F 1 "VCC" H 7400 3650 30  0000 C CNN
 F 2 "" H 7400 3550 60  0000 C CNN
@@
 $EndComp
 $Comp
-L GND-RESCUE-drawdio #PWR08
+L GND-RESCUE-drawdio #PWR07
 U 1 1 558086F5
 P 4600 4550
-F 0 "#PWR08" H 4600 4550 30  0001 C CNN
+F 0 "#PWR07" H 4600 4550 30  0001 C CNN
 F 1 "GND" H 4600 4480 30  0001 C CNN
 F 2 "" H 4600 4550 60  0000 C CNN
@@
 $EndComp
 $Comp
-L VCC #PWR09
+L VCC #PWR08
 U 1 1 55808C03
 P 3650 4250
-F 0 "#PWR09" H 3650 4350 30  0001 C CNN
+F 0 "#PWR08" H 3650 4350 30  0001 C CNN
 F 1 "VCC" H 3650 4350 30  0000 C CNN
 F 2 "" H 3650 4250 60  0000 C CNN
@@
 	4600 4550 4600 4400
 $Comp
-L CONN_01X01 P?
+L CONN_01X01 P2
 U 1 1 55EF137E
 P 8400 4000
-F 0 "P?" H 8400 4100 50  0000 C CNN
+F 0 "P2" H 8400 4100 50  0000 C CNN
 F 1 "CONN_01X01" V 8500 4000 50  0000 C CNN
-F 2 "" H 8400 4000 60  0000 C CNN
+F 2 "Pin_Headers:Pin_Header_Straight_1x01" H 8400 4000 60  0001 C CNN
 F 3 "" H 8400 4000 60  0000 C CNN
 	1    8400 4000
