File: _saved_drawdio.sch (KiCad schematic (older format))
At the start: 15 parts, among them P1 CONN_01X01, P2 CONN_01X02, P3 CONN_01X01, Q1 BC558, Q2 BC547, Q3 BC558, Q4 BC547, U1 LM555N

Commit message: Heavy work
Parts:
- added P3, P5, P6, P7: CONN_01X01, Mounting_Holes:MountingHole_2-5mm, symbol CONN_01X01
- BT1: footprint drawdio:CR2025 Keystone 3002 button cell holder SMT -> drawdio:CR2025_Keystone_3002_button_cell_holder_SMT
- P1: footprint drawdio:Drawdio conn -> drawdio:Drawdio_conn
- P2: renamed from P3; footprint drawdio:Drawdio conn -> drawdio:Drawdio_conn
- P4: renamed from P2; footprint drawdio:RS mini speaker 724-3100 -> drawdio:RS_mini_speaker_724-3100
- Q1: renamed from Q3; footprint drawdio:TO-92_JorFru_compact -> Housings_TO-92:TO-92_Molded_Wide_Oval
- Q2: renamed from Q4; footprint drawdio:TO-92_JorFru_compact -> Housings_TO-92:TO-92_Molded_Wide_Oval
- Q3: renamed from Q1; footprint drawdio:TO-92_JorFru_compact -> Housings_TO-92:TO-92_Molded_Wide_Oval
- Q4: renamed from Q2; footprint drawdio:TO-92_JorFru_compact -> Housings_TO-92:TO-92_Molded_Wide_Oval
Connections:
- no-connect marks 0 -> 4
Changed lines of the file:
@@
 $EndComp
 $Comp
-L BC558 Q1
+L BC558 Q3
 U 1 1 553583B6
 P 7850 3750
-F 0 "Q1" H 7850 3601 40  0000 R CNN
+F 0 "Q3" H 7850 3601 40  0000 R CNN
 F 1 "BC558" H 7850 3900 40  0000 R CNN
-F 2 "drawdio:TO-92_JorFru_compact" H 7750 3852 29  0000 C CNN
+F 2 "Housings_TO-92:TO-92_Molded_Wide_Oval" H 7750 3852 29  0000 C CNN
 F 3 "" H 7850 3750 60  0000 C CNN
 	1    7850 3750
@@
 F 0 "BT1" H 3250 4800 50  0000 C CNN
 F 1 "BATTERY" H 3250 4410 50  0000 C CNN
-F 2 "drawdio:CR2025 Keystone 3002 button cell holder SMT" H 3250 4600 60  0000 C CNN
+F 2 "drawdio:CR2025_Keystone_3002_button_cell_holder_SMT" H 3250 4600 60  0000 C CNN
 F 3 "~" H 3250 4600 60  0000 C CNN
 	1    3250 4600
@@
 F 0 "P1" H 5250 2250 50  0000 C CNN
 F 1 "CONN_01X01" V 5350 2150 50  0000 C CNN
-F 2 "drawdio:Drawdio conn" H 5250 2150 60  0001 C CNN
+F 2 "drawdio:Drawdio_conn" H 5250 2150 60  0001 C CNN
 F 3 "" H 5250 2150 60  0000 C CNN
 	1    5250 2150
@@
 $EndComp
 $Comp
-L CONN_01X01 P3
+L CONN_01X01 P2
 U 1 1 56241E1F
 P 5450 2150
-F 0 "P3" H 5450 2250 50  0000 C CNN
+F 0 "P2" H 5450 2250 50  0000 C CNN
 F 1 "CONN_01X01" V 5550 2150 50  0000 C CNN
-F 2 "drawdio:Drawdio conn" H 5450 2150 60  0001 C CNN
+F 2 "drawdio:Drawdio_conn" H 5450 2150 60  0001 C CNN
 F 3 "" H 5450 2150 60  0000 C CNN
 	1    5450 2150
@@
 $EndComp
 $Comp
-L BC547 Q2
+L BC547 Q4
 U 1 1 553583A7
 P 7850 4250
-F 0 "Q2" H 7850 4101 40  0000 R CNN
+F 0 "Q4" H 7850 4101 40  0000 R CNN
 F 1 "BC547" H 7850 4400 40  0000 R CNN
-F 2 "drawdio:TO-92_JorFru_compact" H 7750 4352 29  0000 C CNN
+F 2 "Housings_TO-92:TO-92_Molded_Wide_Oval" H 7750 4352 29  0000 C CNN
 F 3 "" H 7850 4250 60  0000 C CNN
 	1    7850 4250
@@
 $EndComp
 $Comp
-L BC558 Q3
+L BC558 Q1
 U 1 1 5624397B
 P 7300 3750
-F 0 "Q3" H 7300 3601 40  0000 R CNN
+F 0 "Q1" H 7300 3601 40  0000 R CNN
 F 1 "BC558" H 7300 3900 40  0000 R CNN
-F 2 "drawdio:TO-92_JorFru_compact" H 7200 3852 29  0000 C CNN
+F 2 "Housings_TO-92:TO-92_Molded_Wide_Oval" H 7200 3852 29  0000 C CNN
 F 3 "" H 7300 3750 60  0000 C CNN
 	1    7300 3750
@@
 	7400 4600 7400 4450
 $Comp
-L BC547 Q4
+L BC547 Q2
 U 1 1 56243988
 P 7300 4250
-F 0 "Q4" H 7300 4101 40  0000 R CNN
+F 0 "Q2" H 7300 4101 40  0000 R CNN
 F 1 "BC547" H 7300 4400 40  0000 R CNN
-F 2 "drawdio:TO-92_JorFru_compact" H 7200 4352 29  0000 C CNN
+F 2 "Housings_TO-92:TO-92_Molded_Wide_Oval" H 7200 4352 29  0000 C CNN
 F 3 "" H 7300 4250 60  0000 C CNN
 	1    7300 4250
@@
 Connection ~ 7550 4000
 $Comp
-L CONN_01X02 P2
+L CONN_01X02 P4
 U 1 1 562400DE
 P 8650 4850
-F 0 "P2" H 8650 5000 50  0000 C CNN
+F 0 "P4" H 8650 5000 50  0000 C CNN
 F 1 "CONN_01X02" V 8750 4850 50  0000 C CNN
-F 2 "drawdio:RS mini speaker 724-3100" H 8650 4850 60  0001 C CNN
+F 2 "drawdio:RS_mini_speaker_724-3100" H 8650 4850 60  0001 C CNN
 F 3 "" H 8650 4850 60  0000 C CNN
 	1    8650 4850
 	1    0    0    -1
 $EndComp
+$Comp
+L CONN_01X01 P3
+U 1 1 56244D2E
+P 8300 2600
+F 0 "P3" H 8300 2700 50  0000 C CNN
+F 1 "CONN_01X01" V 8400 2600 50  0000 C CNN
+F 2 "Mounting_Holes:MountingHole_2-5mm" H 8300 2600 60  0001 C CNN
+F 3 "" H 8300 2600 60  0000 C CNN
+	1    8300 2600
+	0    -1   -1   0
+$EndComp
+NoConn ~ 8300 2800
+$Comp
+L CONN_01X01 P5
+U 1 1 56244EEB
+P 8750 2600
+F 0 "P5" H 8750 2700 50  0000 C CNN
+F 1 "CONN_01X01" V 8850 2600 50  0000 C CNN
+F 2 "Mounting_Holes:MountingHole_2-5mm" H 8750 2600 60  0001 C CNN
+F 3 "" H 8750 2600 60  0000 C CNN
+	1    8750 2600
+	0    -1   -1   0
+$EndComp
+NoConn ~ 8750 2800
+$Comp
+L CONN_01X01 P6
+U 1 1 56244F67
+P 9150 2600
+F 0 "P6" H 9150 2700 50  0000 C CNN
+F 1 "CONN_01X01" V 9250 2600 50  0000 C CNN
+F 2 "Mounting_Holes:MountingHole_2-5mm" H 9150 2600 60  0001 C CNN
+F 3 "" H 9150 2600 60  0000 C CNN
+	1    9150 2600
+	0    -1   -1   0
+$EndComp
+NoConn ~ 9150 2800
+$Comp
+L CONN_01X01 P7
+U 1 1 56244F6E
+P 9600 2600
+F 0 "P7" H 9600 2700 50  0000 C CNN
+F 1 "CONN_01X01" V 9700 2600 50  0000 C CNN
+F 2 "Mounting_Holes:MountingHole_2-5mm" H 9600 2600 60  0001 C CNN
+F 3 "" H 9600 2600 60  0000 C CNN
+	1    9600 2600
+	0    -1   -1   0
+$EndComp
+NoConn ~ 9600 2800
 $EndSCHEMATC
