File: KiCad files/drawdio.sch (KiCad schematic (older format))
At the start: 23 parts, among them P1 CONN_01X01, P10 CONN_01X02, P2 CONN_01X01, P3 CONN_01X01, P4 CONN_01X02, P5 CONN_01X01, P6 CONN_01X01, P7 CONN_01X01, P9 CONN_02X04, Q1 BC558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

Commit message: schematic upgrades
Parts:
- removed P10: CONN_01X02, drawdio:AAA_cell_holder, symbol CONN_01X02
- removed P3, P5, P6, P7: CONN_01X01, Mounting_Holes:MountingHole_2-5mm, symbol CONN_01X01
- added J1: Jack, symbol JACK_TRS_6PINS
- added P3: PWR_SW, symbol CONN_01X03
- C1, C4: value CP -> 470uF
- C2: value C -> 0.1uF
- C3: value C -> 680pF
- P1: value CONN_01X01 -> CON1
- P2: value CONN_01X01 -> CON2
- P4: value CONN_01X02 -> SPK
- R1: value R -> 330K
- R2: value R -> 10K
- R3, R4: value R -> 1K
- U1: symbol LM555N -> LM555N-RESCUE-drawdio
Connections:
- wire segments 36 -> 42
Other:
- note added: "Salida jack"
- note removed: "Taladros mecánicos"
- moved on the sheet: BT1, C1, R2

Commit message: Checkpoint, a dormir!
Parts:
- removed U1: LM555N, Housings_DIP:DIP-8_W7.62mm_LongPads, symbol LM555N-RESCUE-drawdio
- added U1: NE555, Housings_DIP:DIP-8_W7.62mm_Socket_LongPads, symbol NE555
- BT1: footprint drawdio:CR2025_Keystone_3002_button_cell_holder_SMT -> drawdio:AAA_cell_holder
- C2, R1, R2: footprint Discret:R3 -> Resistors_Universal:Resistor_SMD+THTuniversal_0805to1206_RM10_HandSoldering
- C3: footprint Capacitors_ThroughHole:C_Rect_L4_W2.5_P2.5 -> Resistors_Universal:Resistor_SMD+THTuniversal_0805to1206_RM10_HandSoldering
- J1: footprint (none) -> Connect:BARREL_JACK
- P3: footprint (none) -> drawdio:PWR_SW_Drawdio_SS-12D00(1P2T)
- Q1, Q2, Q3, Q4: footprint Housings_TO-92:TO-92_Molded_Wide_Oval -> drawdio:TO-92_JorFru_compact
- R3, R4: footprint Discret:R1 -> Resistors_Universal:Resistor_SMD+THTuniversal_0805to1206_RM10_HandSoldering
Other:
- moved on the sheet: C2
Changed lines of the file:
@@
 LIBS:contrib
 LIBS:valves
-LIBS:kicad-library
 LIBS:drawdio-cache
 EELAYER 25 0
@@
 $EndDescr
 $Comp
-L LM555N-RESCUE-drawdio U1
-U 1 1 55357FC1
-P 5600 3950
-F 0 "U1" H 5600 4050 70  0000 C CNN
-F 1 "LM555N" H 5600 3850 70  0000 C CNN
-F 2 "Housings_DIP:DIP-8_W7.62mm_LongPads" H 5600 3950 60  0001 C CNN
-F 3 "" H 5600 3950 60  0000 C CNN
-	1    5600 3950
-	1    0    0    -1
-$EndComp
-$Comp
 L R-RESCUE-drawdio R1
 U 1 1 55358209
@@
 F 0 "R1" V 4730 3000 40  0000 C CNN
 F 1 "330K" V 4657 3001 40  0000 C CNN
-F 2 "Discret:R3" V 4580 3000 30  0000 C CNN
+F 2 "Resistors_Universal:Resistor_SMD+THTuniversal_0805to1206_RM10_HandSoldering" V 4580 3000 30  0000 C CNN
 F 3 "~" H 4650 3000 30  0000 C CNN
 	1    4650 3000
@@
 F 0 "R2" V 6430 3000 40  0000 C CNN
 F 1 "10K" V 6357 3001 40  0000 C CNN
-F 2 "Discret:R3" V 6280 3000 30  0000 C CNN
+F 2 "Resistors_Universal:Resistor_SMD+THTuniversal_0805to1206_RM10_HandSoldering" V 6280 3000 30  0000 C CNN
 F 3 "~" H 6350 3000 30  0000 C CNN
 	1    6350 3000
@@
 L C-RESCUE-drawdio C2
 U 1 1 55358310
-P 4600 4200
-F 0 "C2" H 4600 4300 40  0000 L CNN
-F 1 "0.1uF" H 4606 4115 40  0000 L CNN
-F 2 "Discret:R3" H 4638 4050 30  0000 C CNN
-F 3 "~" H 4600 4200 60  0000 C CNN
-	1    4600 4200
+P 4800 4150
+F 0 "C2" H 4800 4250 40  0000 L CNN
+F 1 "0.1uF" H 4806 4065 40  0000 L CNN
+F 2 "Resistors_Universal:Resistor_SMD+THTuniversal_0805to1206_RM10_HandSoldering" H 4838 4000 30  0000 C CNN
+F 3 "~" H 4800 4150 60  0000 C CNN
+	1    4800 4150
 	1    0    0    -1
 $EndComp
@@
 L VCC #PWR02
 U 1 1 55358356
-P 4800 4250
-F 0 "#PWR02" H 4800 4350 30  0001 C CNN
-F 1 "VCC" H 4800 4350 30  0000 C CNN
-F 2 "" H 4800 4250 60  0000 C CNN
-F 3 "" H 4800 4250 60  0000 C CNN
-	1    4800 4250
+P 5000 4150
+F 0 "#PWR02" H 5000 4250 30  0001 C CNN
+F 1 "VCC" H 5000 4250 30  0000 C CNN
+F 2 "" H 5000 4150 60  0000 C CNN
+F 3 "" H 5000 4150 60  0000 C CNN
+	1    5000 4150
 	1    0    0    -1
 $EndComp
@@
 F 0 "Q3" H 8350 3351 40  0000 R CNN
 F 1 "BC558" H 8350 3650 40  0000 R CNN
-F 2 "Housings_TO-92:TO-92_Molded_Wide_Oval" H 7700 3600 29  0001 C CNN
+F 2 "drawdio:TO-92_JorFru_compact" H 7700 3600 29  0001 C CNN
 F 3 "" H 8350 3500 60  0000 C CNN
 	1    8350 3500
@@
 F 0 "C3" H 6550 5300 40  0000 L CNN
 F 1 "680pF" H 6556 5115 40  0000 L CNN
-F 2 "Capacitors_ThroughHole:C_Rect_L4_W2.5_P2.5" H 6588 5050 30  0001 C CNN
+F 2 "Resistors_Universal:Resistor_SMD+THTuniversal_0805to1206_RM10_HandSoldering" H 6588 5050 30  0001 C CNN
 F 3 "~" H 6550 5200 60  0000 C CNN
 	1    6550 5200
@@
 F 0 "BT1" H 2650 4800 50  0000 C CNN
 F 1 "BATTERY" H 2650 4410 50  0000 C CNN
-F 2 "drawdio:CR2025_Keystone_3002_button_cell_holder_SMT" H 2800 5350 60  0001 C CNN
+F 2 "drawdio:AAA_cell_holder" H 2800 5350 60  0001 C CNN
 F 3 "~" H 2650 4600 60  0000 C CNN
 	1    2650 4600
@@
 L GND-RESCUE-drawdio #PWR07
 U 1 1 558086F5
-P 4600 4550
-F 0 "#PWR07" H 4600 4550 30  0001 C CNN
-F 1 "GND" H 4600 4480 30  0001 C CNN
-F 2 "" H 4600 4550 60  0000 C CNN
-F 3 "" H 4600 4550 60  0000 C CNN
-	1    4600 4550
+P 4800 4500
+F 0 "#PWR07" H 4800 4500 30  0001 C CNN
+F 1 "GND" H 4800 4430 30  0001 C CNN
+F 2 "" H 4800 4500 60  0000 C CNN
+F 3 "" H 4800 4500 60  0000 C CNN
+	1    4800 4500
 	1    0    0    -1
 $EndComp
@@
 F 0 "Q4" H 8350 3851 40  0000 R CNN
 F 1 "BC547" H 8350 4150 40  0000 R CNN
-F 2 "Housings_TO-92:TO-92_Molded_Wide_Oval" H 8250 4102 29  0001 C CNN
+F 2 "drawdio:TO-92_JorFru_compact" H 8250 4102 29  0001 C CNN
 F 3 "" H 8350 4000 60  0000 C CNN
 	1    8350 4000
@@
 F 0 "Q1" H 7450 3351 40  0000 R CNN
 F 1 "BC558" H 7450 3650 40  0000 R CNN
-F 2 "Housings_TO-92:TO-92_Molded_Wide_Oval" H 7350 3602 29  0001 C CNN
+F 2 "drawdio:TO-92_JorFru_compact" H 7350 3602 29  0001 C CNN
 F 3 "" H 7450 3500 60  0000 C CNN
 	1    7450 3500
@@
 F 0 "Q2" H 7450 3851 40  0000 R CNN
 F 1 "BC547" H 7450 4150 40  0000 R CNN
-F 2 "Housings_TO-92:TO-92_Molded_Wide_Oval" V 7350 4102 29  0001 C CNN
+F 2 "drawdio:TO-92_JorFru_compact" V 7350 4102 29  0001 C CNN
 F 3 "" H 7450 4000 60  0000 C CNN
 	1    7450 4000
@@
 Text Label 6300 4150 1    60   ~ 0
 pin6
-Text Label 4900 4250 1    60   ~ 0
+Text Label 5100 4150 1    60   ~ 0
 pin4
-Text Label 4900 4000 1    60   ~ 0
+Text Label 5100 3950 1    60   ~ 0
 pin5
 $Comp
@@
 F 0 "R4" V 8080 3750 50  0000 C CNN
 F 1 "1K" V 8000 3750 50  0000 C CNN
-F 2 "Discret:R1" V 7930 3750 30  0001 C CNN
+F 2 "Resistors_Universal:Resistor_SMD+THTuniversal_0805to1206_RM10_HandSoldering" V 7930 3750 30  0001 C CNN
 F 3 "" H 8000 3750 30  0000 C CNN
 	1    8000 3750
@@
 F 0 "R3" V 7080 3750 50  0000 C CNN
 F 1 "1K" V 7000 3750 50  0000 C CNN
-F 2 "Discret:R1" V 6930 3750 30  0001 C CNN
+F 2 "Resistors_Universal:Resistor_SMD+THTuniversal_0805to1206_RM10_HandSoldering" V 6930 3750 30  0001 C CNN
 F 3 "" H 7000 3750 30  0000 C CNN
 	1    7000 3750
@@
 F 0 "J1" H 8850 6050 50  0000 C CNN
 F 1 "Jack" H 8800 5350 50  0000 C CNN
-F 2 "" H 8950 5500 50  0000 C CNN
+F 2 "Connect:BARREL_JACK" H 8950 5500 50  0001 C CNN
 F 3 "" H 8950 5500 50  0000 C CNN
 	1    8850 5650
@@
 F 0 "P3" H 3150 4750 50  0000 C CNN
 F 1 "PWR_SW" V 3250 4550 50  0000 C CNN
-F 2 "" H 3150 4550 50  0000 C CNN
+F 2 "drawdio:PWR_SW_Drawdio_SS-12D00(1P2T)" H 3150 4550 50  0001 C CNN
 F 3 "" H 3150 4550 50  0000 C CNN
 	1    3150 4550
@@
 NoConn ~ 3050 4350
 Wire Wire Line
-	4400 3750 4900 3750
+	4400 3750 5100 3750
 Wire Wire Line
 	4650 3750 4650 3250
@@
 	6550 4150 6550 5000
 Wire Wire Line
-	6550 4150 6300 4150
+	6100 4150 6550 4150
 Connection ~ 4650 3750
 Wire Wire Line
-	6550 2750 6550 3950
-Wire Wire Line
-	6550 3950 6300 3950
+	6550 3950 6550 2750
+Wire Wire Line
+	6100 3950 6550 3950
 Wire Wire Line
 	8450 4350 8450 4200
 Wire Wire Line
-	4600 4000 4900 4000
-Wire Wire Line
-	4800 4250 4900 4250
+	4800 3950 5100 3950
 Wire Wire Line
 	6450 3250 6350 3250
@@
 Connection ~ 3600 4900
 Wire Wire Line
-	4600 4550 4600 4400
+	4800 4500 4800 4350
 Wire Wire Line
 	7550 4350 7550 4200
@@
 Connection ~ 7250 3750
 Wire Wire Line
-	6300 3750 6850 3750
+	6100 3750 6850 3750
 Wire Wire Line
 	7150 3750 7250 3750
@@
 	8300 4850 8800 4850
 Connection ~ 8800 4850
+$Comp
+L NE555 U1
+U 1 1 5884E805
+P 5600 3950
+F 0 "U1" H 5200 4300 50  0000 L CNN
+F 1 "NE555" H 5200 3600 50  0000 L CNN
+F 2 "Housings_DIP:DIP-8_W7.62mm_Socket_LongPads" H 5600 3950 50  0001 C CNN
+F 3 "" H 5600 3950 50  0000 C CNN
+	1    5600 3950
+	1    0    0    -1
+$EndComp
+Wire Wire Line
+	5100 4150 5000 4150
 $EndSCHEMATC

Commit message: Redimensionada
Parts:
- C2, C3, R1, R2, R3, R4: footprint Resistors_Universal:Resistor_SMD+THTuniversal_0805to1206_RM10_HandSoldering -> drawdio:Resistor_SMD+THTuniversal_0805to1206_RM10_HandSoldering
- J1: footprint Connect:BARREL_JACK -> drawdio:jack_barato
Changed lines of the file:
@@
 F 0 "R1" V 4730 3000 40  0000 C CNN
 F 1 "330K" V 4657 3001 40  0000 C CNN
-F 2 "Resistors_Universal:Resistor_SMD+THTuniversal_0805to1206_RM10_HandSoldering" V 4580 3000 30  0000 C CNN
+F 2 "drawdio:Resistor_SMD+THTuniversal_0805to1206_RM10_HandSoldering" V 4580 3000 30  0000 C CNN
 F 3 "~" H 4650 3000 30  0000 C CNN
 	1    4650 3000
@@
 F 0 "R2" V 6430 3000 40  0000 C CNN
 F 1 "10K" V 6357 3001 40  0000 C CNN
-F 2 "Resistors_Universal:Resistor_SMD+THTuniversal_0805to1206_RM10_HandSoldering" V 6280 3000 30  0000 C CNN
+F 2 "drawdio:Resistor_SMD+THTuniversal_0805to1206_RM10_HandSoldering" V 6280 3000 30  0000 C CNN
 F 3 "~" H 6350 3000 30  0000 C CNN
 	1    6350 3000
@@
 F 0 "C2" H 4800 4250 40  0000 L CNN
 F 1 "0.1uF" H 4806 4065 40  0000 L CNN
-F 2 "Resistors_Universal:Resistor_SMD+THTuniversal_0805to1206_RM10_HandSoldering" H 4838 4000 30  0000 C CNN
+F 2 "drawdio:Resistor_SMD+THTuniversal_0805to1206_RM10_HandSoldering" H 4838 4000 30  0000 C CNN
 F 3 "~" H 4800 4150 60  0000 C CNN
 	1    4800 4150
@@
 F 0 "C3" H 6550 5300 40  0000 L CNN
 F 1 "680pF" H 6556 5115 40  0000 L CNN
-F 2 "Resistors_Universal:Resistor_SMD+THTuniversal_0805to1206_RM10_HandSoldering" H 6588 5050 30  0001 C CNN
+F 2 "drawdio:Resistor_SMD+THTuniversal_0805to1206_RM10_HandSoldering" H 6588 5050 30  0001 C CNN
 F 3 "~" H 6550 5200 60  0000 C CNN
 	1    6550 5200
@@
 F 0 "R4" V 8080 3750 50  0000 C CNN
 F 1 "1K" V 8000 3750 50  0000 C CNN
-F 2 "Resistors_Universal:Resistor_SMD+THTuniversal_0805to1206_RM10_HandSoldering" V 7930 3750 30  0001 C CNN
+F 2 "drawdio:Resistor_SMD+THTuniversal_0805to1206_RM10_HandSoldering" V 7930 3750 30  0001 C CNN
 F 3 "" H 8000 3750 30  0000 C CNN
 	1    8000 3750
@@
 F 0 "R3" V 7080 3750 50  0000 C CNN
 F 1 "1K" V 7000 3750 50  0000 C CNN
-F 2 "Resistors_Universal:Resistor_SMD+THTuniversal_0805to1206_RM10_HandSoldering" V 6930 3750 30  0001 C CNN
+F 2 "drawdio:Resistor_SMD+THTuniversal_0805to1206_RM10_HandSoldering" V 6930 3750 30  0001 C CNN
 F 3 "" H 7000 3750 30  0000 C CNN
 	1    7000 3750
@@
 F 0 "J1" H 8850 6050 50  0000 C CNN
 F 1 "Jack" H 8800 5350 50  0000 C CNN
-F 2 "Connect:BARREL_JACK" H 8950 5500 50  0001 C CNN
+F 2 "drawdio:jack_barato" H 8950 5500 50  0001 C CNN
 F 3 "" H 8950 5500 50  0000 C CNN
 	1    8850 5650

Commit message: puede que funcione
Parts:
- C2, C3, R1, R2, R3, R4: footprint drawdio:Resistor_SMD+THTuniversal_0805to1206_RM10_HandSoldering -> drawdio:Resistor_SMD+THT
Changed lines of the file:
@@
 F 0 "R1" V 4730 3000 40  0000 C CNN
 F 1 "330K" V 4657 3001 40  0000 C CNN
-F 2 "drawdio:Resistor_SMD+THTuniversal_0805to1206_RM10_HandSoldering" V 4580 3000 30  0000 C CNN
+F 2 "drawdio:Resistor_SMD+THT" V 4580 3000 30  0000 C CNN
 F 3 "~" H 4650 3000 30  0000 C CNN
 	1    4650 3000
@@
 F 0 "R2" V 6430 3000 40  0000 C CNN
 F 1 "10K" V 6357 3001 40  0000 C CNN
-F 2 "drawdio:Resistor_SMD+THTuniversal_0805to1206_RM10_HandSoldering" V 6280 3000 30  0000 C CNN
+F 2 "drawdio:Resistor_SMD+THT" V 6280 3000 30  0000 C CNN
 F 3 "~" H 6350 3000 30  0000 C CNN
 	1    6350 3000
@@
 F 0 "C2" H 4800 4250 40  0000 L CNN
 F 1 "0.1uF" H 4806 4065 40  0000 L CNN
-F 2 "drawdio:Resistor_SMD+THTuniversal_0805to1206_RM10_HandSoldering" H 4838 4000 30  0000 C CNN
+F 2 "drawdio:Resistor_SMD+THT" H 4838 4000 30  0000 C CNN
 F 3 "~" H 4800 4150 60  0000 C CNN
 	1    4800 4150
@@
 F 0 "C3" H 6550 5300 40  0000 L CNN
 F 1 "680pF" H 6556 5115 40  0000 L CNN
-F 2 "drawdio:Resistor_SMD+THTuniversal_0805to1206_RM10_HandSoldering" H 6588 5050 30  0001 C CNN
+F 2 "drawdio:Resistor_SMD+THT" H 6588 5050 30  0001 C CNN
 F 3 "~" H 6550 5200 60  0000 C CNN
 	1    6550 5200
@@
 F 0 "R4" V 8080 3750 50  0000 C CNN
 F 1 "1K" V 8000 3750 50  0000 C CNN
-F 2 "drawdio:Resistor_SMD+THTuniversal_0805to1206_RM10_HandSoldering" V 7930 3750 30  0001 C CNN
+F 2 "drawdio:Resistor_SMD+THT" V 7930 3750 30  0001 C CNN
 F 3 "" H 8000 3750 30  0000 C CNN
 	1    8000 3750
@@
 F 0 "R3" V 7080 3750 50  0000 C CNN
 F 1 "1K" V 7000 3750 50  0000 C CNN
-F 2 "drawdio:Resistor_SMD+THTuniversal_0805to1206_RM10_HandSoldering" V 6930 3750 30  0001 C CNN
+F 2 "drawdio:Resistor_SMD+THT" V 6930 3750 30  0001 C CNN
 F 3 "" H 7000 3750 30  0000 C CNN
 	1    7000 3750
@@
 $EndComp
 NoConn ~ 3050 4350
-Wire Wire Line
-	4400 3750 5100 3750
-Wire Wire Line
-	4650 3750 4650 3250
-Wire Wire Line
-	5250 2750 5250 2350
-Wire Wire Line
-	4400 3750 4400 4900
-Wire Wire Line
-	4400 4900 6550 4900
-Wire Wire Line
-	6550 4150 6550 5000
-Wire Wire Line
-	6100 4150 6550 4150
-Connection ~ 4650 3750
-Wire Wire Line
-	6550 3950 6550 2750
-Wire Wire Line
-	6100 3950 6550 3950
-Wire Wire Line
-	8450 4350 8450 4200
-Wire Wire Line
-	4800 3950 5100 3950
-Wire Wire Line
-	6450 3250 6350 3250
-Wire Wire Line
-	6550 5550 6550 5400
-Connection ~ 6550 4900
-Wire Wire Line
-	4650 2750 5250 2750
-Wire Wire Line
-	5450 2350 5450 2750
-Wire Wire Line
-	5450 2750 6550 2750
-Wire Wire Line
-	3600 4250 3600 4400
-Wire Wire Line
-	3600 4800 3600 5050
-Connection ~ 3600 4300
-Connection ~ 3600 4900
-Wire Wire Line
-	4800 4500 4800 4350
-Wire Wire Line
-	7550 4350 7550 4200
-Wire Wire Line
-	7250 3500 7250 4000
-Wire Wire Line
-	7550 3700 7550 3800
-Wire Wire Line
-	8150 3500 8150 4000
-Connection ~ 7550 3750
-Connection ~ 8150 3750
-Wire Wire Line
-	8800 4150 8800 5000
-Wire Wire Line
-	8450 3700 8450 3800
-Connection ~ 8450 3750
-Wire Wire Line
-	7700 5100 8800 5100
-Connection ~ 7700 3750
-Wire Wire Line
-	8450 3750 8800 3750
-Wire Wire Line
-	7550 3750 7850 3750
-Connection ~ 7250 3750
-Wire Wire Line
-	6100 3750 6850 3750
-Wire Wire Line
-	7150 3750 7250 3750
-Wire Notes Line
-	6800 3050 6800 4450
-Wire Notes Line
-	6800 4450 9050 4450
-Wire Notes Line
-	9050 4450 9050 3050
-Wire Notes Line
-	9050 3050 6800 3050
-Wire Notes Line
-	4900 1850 4900 2400
-Wire Notes Line
-	4900 2400 5850 2400
-Wire Notes Line
-	5850 2400 5850 1850
-Wire Notes Line
-	5850 1850 4900 1850
-Wire Notes Line
-	4250 2550 4250 5650
-Wire Notes Line
-	4250 5650 6700 5650
-Wire Notes Line
-	6700 5650 6700 2550
-Wire Notes Line
-	6700 2550 4250 2550
-Wire Notes Line
-	5050 2800 5050 3300
-Wire Notes Line
-	5050 3300 6050 3300
-Wire Notes Line
-	6050 3300 6050 2800
-Wire Notes Line
-	6050 2800 5050 2800
-Wire Wire Line
-	2650 4900 3600 4900
-Connection ~ 7700 5100
-Wire Wire Line
-	8300 5450 8450 5450
-Wire Wire Line
-	8300 5650 8450 5650
-Connection ~ 8300 5450
-Wire Wire Line
-	8450 5850 7700 5850
-Wire Wire Line
-	7700 5850 7700 3750
-Wire Wire Line
-	3600 4300 3250 4300
-Wire Wire Line
-	3250 4300 3250 4350
-Wire Wire Line
-	3150 4350 3150 4300
-Wire Wire Line
-	3150 4300 2650 4300
-Connection ~ 3350 4300
-Connection ~ 3350 4900
-Wire Notes Line
-	3900 4050 3900 5150
-Wire Notes Line
-	3900 5150 2400 5150
-Wire Notes Line
-	2400 5150 2400 4050
-Wire Notes Line
-	2400 4050 3900 4050
-Connection ~ 6350 2750
-Wire Notes Line
-	9950 6100 7550 6100
-Wire Notes Line
-	7550 6100 7550 4700
-Wire Notes Line
-	7550 4700 9950 4700
-Wire Notes Line
-	9950 4700 9950 6100
-Wire Wire Line
-	8300 5650 8300 4850
-Wire Wire Line
-	8300 4850 8800 4850
-Connection ~ 8800 4850
 $Comp
 L NE555 U1
@@
 $EndComp
 Wire Wire Line
+	4400 3750 5100 3750
+Wire Wire Line
+	4650 3750 4650 3250
+Wire Wire Line
+	5250 2750 5250 2350
+Wire Wire Line
+	4400 3750 4400 4900
+Wire Wire Line
+	4400 4900 6550 4900
+Wire Wire Line
+	6550 4150 6550 5000
+Wire Wire Line
+	6100 4150 6550 4150
+Connection ~ 4650 3750
+Wire Wire Line
+	6550 3950 6550 2750
+Wire Wire Line
+	6100 3950 6550 3950
+Wire Wire Line
+	8450 4350 8450 4200
+Wire Wire Line
+	4800 3950 5100 3950
+Wire Wire Line
+	6450 3250 6350 3250
+Wire Wire Line
+	6550 5550 6550 5400
+Connection ~ 6550 4900
+Wire Wire Line
+	4650 2750 5250 2750
+Wire Wire Line
+	5450 2350 5450 2750
+Wire Wire Line
+	5450 2750 6550 2750
+Wire Wire Line
+	3600 4250 3600 4400
+Wire Wire Line
+	3600 4800 3600 5050
+Connection ~ 3600 4300
+Connection ~ 3600 4900
+Wire Wire Line
+	4800 4500 4800 4350
+Wire Wire Line
+	7550 4350 7550 4200
+Wire Wire Line
+	7250 3500 7250 4000
+Wire Wire Line
+	7550 3700 7550 3800
+Wire Wire Line
+	8150 3500 8150 4000
+Connection ~ 7550 3750
+Connection ~ 8150 3750
+Wire Wire Line
+	8800 4150 8800 5000
+Wire Wire Line
+	8450 3700 8450 3800
+Connection ~ 8450 3750
+Wire Wire Line
+	7700 5100 8800 5100
+Connection ~ 7700 3750
+Wire Wire Line
+	8450 3750 8800 3750
+Wire Wire Line
+	7550 3750 7850 3750
+Connection ~ 7250 3750
+Wire Wire Line
+	6100 3750 6850 3750
+Wire Wire Line
+	7150 3750 7250 3750
+Wire Notes Line
+	6800 3050 6800 4450
+Wire Notes Line
+	6800 4450 9050 4450
+Wire Notes Line
+	9050 4450 9050 3050
+Wire Notes Line
+	9050 3050 6800 3050
+Wire Notes Line
+	4900 1850 4900 2400
+Wire Notes Line
+	4900 2400 5850 2400
+Wire Notes Line
+	5850 2400 5850 1850
+Wire Notes Line
+	5850 1850 4900 1850
+Wire Notes Line
+	4250 2550 4250 5650
+Wire Notes Line
+	4250 5650 6700 5650
+Wire Notes Line
+	6700 5650 6700 2550
+Wire Notes Line
+	6700 2550 4250 2550
+Wire Notes Line
+	5050 2800 5050 3300
+Wire Notes Line
+	5050 3300 6050 3300
+Wire Notes Line
+	6050 3300 6050 2800
+Wire Notes Line
+	6050 2800 5050 2800
+Connection ~ 7700 5100
+Wire Wire Line
+	8300 5450 8450 5450
+Wire Wire Line
+	8300 5650 8450 5650
+Connection ~ 8300 5450
+Wire Wire Line
+	8450 5850 7700 5850
+Wire Wire Line
+	7700 5850 7700 3750
+Connection ~ 3350 4300
+Connection ~ 3350 4900
+Wire Notes Line
+	3900 4050 3900 5150
+Wire Notes Line
+	3900 5150 2400 5150
+Wire Notes Line
+	2400 5150 2400 4050
+Wire Notes Line
+	2400 4050 3900 4050
+Connection ~ 6350 2750
+Wire Notes Line
+	9950 6100 7550 6100
+Wire Notes Line
+	7550 6100 7550 4700
+Wire Notes Line
+	7550 4700 9950 4700
+Wire Notes Line
+	9950 4700 9950 6100
+Wire Wire Line
+	8300 5650 8300 4850
+Wire Wire Line
+	8300 4850 8800 4850
+Connection ~ 8800 4850
+Wire Wire Line
 	5100 4150 5000 4150
+Wire Wire Line
+	2650 4900 3600 4900
+Wire Wire Line
+	3250 4300 3250 4350
+Wire Wire Line
+	3600 4300 3250 4300
+Wire Wire Line
+	3150 4350 3150 4300
+Wire Wire Line
+	3150 4300 2650 4300
 $EndSCHEMATC
