File: KiCad files/_saved_drawdio.sch (KiCad schematic (older format))
At the start: 19 parts, among them J1 Jack, P1 CON1, P2 CON2, P3 PWR_SW, P4 SPK, Q1 BC558, Q2 BC547, Q3 BC558, Q4 BC547, U1 NE555

Commit message: Casi terminado
Parts:
- U1: footprint Housings_DIP:DIP-8_W7.62mm_Socket_LongPads -> KiCad_Files:DIP8+SOIC8_2
Changed lines of the file:
@@
 F 0 "U1" H 5200 4300 50  0000 L CNN
 F 1 "NE555" H 5200 3600 50  0000 L CNN
-F 2 "Housings_DIP:DIP-8_W7.62mm_Socket_LongPads" H 5600 3950 50  0001 C CNN
+F 2 "KiCad_Files:DIP8+SOIC8_2" H 5600 3950 50  0001 C CNN
 F 3 "" H 5600 3950 50  0000 C CNN
 	1    5600 3950
