File: KiCad files/drawdio.kicad_pcb (KiCad board)
At the start: 2 copper layers, 90.8 x 22.9 mm, 29 parts, among them J1 Jack, P1 CON1, P2 CON2, P4 SPK

Commit message: presentable V2.0
Parts:
- Q1, Q3: renamed from PNP; footprint drawdio:TO-92_JorFru_compact -> drawdio:TO-92_SOT23_JorFru_compact
- Q2, Q4: renamed from NPN; footprint drawdio:TO-92_JorFru_compact -> drawdio:TO-92_SOT23_JorFru_compact
- moved REF** 1.42 mm to (79.8, 95.9)
- moved REF** 1.42 mm to (79.8, 84.5)
- moved G*** 1.37 mm to (80.4, 90.2)
- moved G*** 1.28 mm to (133.6, 89.5)
- moved REF** 1.27 mm to (134.4, 95.9)
- moved REF** 1.27 mm to (134.4, 84.5)
- renumbered 470uF to C1, 0.1uF to C2, 680pF to C3, 470uF to C4, 330K to R1, 10K to R2, 1K to R3, 1K to R4, 555CMOS to U1

Commit message: Retocado el tamaño de algunas silkscreen
Parts:
- added G***: LOGO, uc3music_logos:logo_pick_6x6mm, B.Cu at (78.4, 79.1)
- G***: moved to B.Cu
- moved G*** 63.0 mm to (71.5, 79.0), turned to 180 degrees
- moved G*** 0.13 mm to (58.3, 87.0)
